File: dac-001s.kicad_pcb (KiCad board)
At the start: 2 copper layers, 70 x 50 mm, 29 parts, among them J1 Conn_01x02, J2 Conn_01x03, J3 Conn_01x06, U1 ADP3338AKCZ-3.3RL7, U2 PCM5102A

Commit message: Added GBR files
Routing:
- net GNDD: track 23.8 -> 20.9 mm
- net GNDA: track 13.2 -> 16.1 mm, vias 13 -> 14
